File: MB-RL7021-11-M5StickC.kicad_sch (KiCad schematic)
At the start: 7 parts, among them J1 Conn_01x08, U1 MB-RL7021-11

Commit message: ver1.1 ねじをm2に変更
Parts:
- H1, H2, H3, H4: footprint MountingHole:MountingHole_3.2mm_M3 -> MountingHole:MountingHole_2.2mm_M2
Changed lines of the file:
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@@
       (effects (font (size 1.27 1.27)) (justify left))
     )
-    (property "Footprint" "MountingHole:MountingHole_3.2mm_M3" (id 2) (at 157.48 166.37 0)
+    (property "Footprint" "MountingHole:MountingHole_2.2mm_M2" (id 2) (at 157.48 166.37 0)
       (effects (font (size 1.27 1.27)) hide)
     )
@@
       (effects (font (size 1.27 1.27)) (justify left))
     )
-    (property "Footprint" "MountingHole:MountingHole_3.2mm_M3" (id 2) (at 135.89 166.37 0)
+    (property "Footprint" "MountingHole:MountingHole_2.2mm_M2" (id 2) (at 135.89 166.37 0)
       (effects (font (size 1.27 1.27)) hide)
     )
@@
       (effects (font (size 1.27 1.27)) (justify left))
     )
-    (property "Footprint" "MountingHole:MountingHole_3.2mm_M3" (id 2) (at 157.48 156.21 0)
+    (property "Footprint" "MountingHole:MountingHole_2.2mm_M2" (id 2) (at 157.48 156.21 0)
       (effects (font (size 1.27 1.27)) hide)
     )
@@
       (effects (font (size 1.27 1.27)) (justify left))
     )
-    (property "Footprint" "MountingHole:MountingHole_3.2mm_M3" (id 2) (at 135.89 156.21 0)
+    (property "Footprint" "MountingHole:MountingHole_2.2mm_M2" (id 2) (at 135.89 156.21 0)
       (effects (font (size 1.27 1.27)) hide)
     )
@@
     )
     (path "/cf2cdba0-73d6-4b66-a4c1-463ebe157ed1"
-      (reference "H1") (unit 1) (value "MountingHole") (footprint "MountingHole:MountingHole_3.2mm_M3")
+      (reference "H1") (unit 1) (value "MountingHole") (footprint "MountingHole:MountingHole_2.2mm_M2")
     )
     (path "/74ee0542-f863-4a3a-bcbb-6820d230aeef"
-      (reference "H2") (unit 1) (value "MountingHole") (footprint "MountingHole:MountingHole_3.2mm_M3")
+      (reference "H2") (unit 1) (value "MountingHole") (footprint "MountingHole:MountingHole_2.2mm_M2")
     )
     (path "/c5c658c6-0ebc-4b64-98c6-e56544d9e547"
-      (reference "H3") (unit 1) (value "MountingHole") (footprint "MountingHole:MountingHole_3.2mm_M3")
+      (reference "H3") (unit 1) (value "MountingHole") (footprint "MountingHole:MountingHole_2.2mm_M2")
     )
     (path "/46c65a1b-07ae-4560-9eb2-734ef1764e37"
-      (reference "H4") (unit 1) (value "MountingHole") (footprint "MountingHole:MountingHole_3.2mm_M3")
+      (reference "H4") (unit 1) (value "MountingHole") (footprint "MountingHole:MountingHole_2.2mm_M2")
     )
     (path "/b1a5f699-e7ea-44f1-ada4-5893a1552b3d"
